File: pcb/batterymonitor-electron.kicad_pcb (KiCad board)
At the start: 2 copper layers, 69 parts, among them M1 particle_electron, P1 CONN_02X10, Q1 Q_NMOS_GSD, Q2 Q_NMOS_GSD, Q3 Q_NMOS_GSD, Q4 Q_NMOS_GSD, Q5 Q_PMOS_GDS, Q6 Q_PMOS_GDS, Q7 Q_PMOS_GDS, Q8 Q_PMOS_GDS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

Commit message: added pcb cuts
Parts:
- removed C10, C3, C4, C5, C6, C7, C8, C9: 0.01uF, Capacitors_SMD:C_0603_HandSoldering
- removed D1, D2, D3, D4: BAV199-7-F, TO_SOT_Packages_SMD:SOT-23_Handsoldering
- removed Q5, Q6, Q7, Q8: Q_PMOS_GDS, TO_SOT_Packages_SMD:TO-263-3Lead
- removed R17, R18, R19, R20, R21, R22, R23, R24: 100R, Resistors_SMD:R_0603_HandSoldering
- removed R41, R42, R43, R44: R, Resistors_SMD:R_0603_HandSoldering
- added M2: R-78E-0.5, TO_SOT_Packages_THT:TO-220_Vertical, F.Cu at (106.0, 102.5)
- added REF**: MountingHole_3.2mm_M3_DIN965, Mounting_Holes:MountingHole_3.2mm_M3_DIN965, F.Cu at (75.0, 69.8)
- added REF**: MountingHole_3.2mm_M3_DIN965, Mounting_Holes:MountingHole_3.2mm_M3_DIN965, F.Cu at (125.0, 69.8)
- added REF**: MountingHole_3.2mm_M3_DIN965, Mounting_Holes:MountingHole_3.2mm_M3_DIN965, F.Cu at (75.0, 130.2)
- added REF**: MountingHole_3.2mm_M3_DIN965, Mounting_Holes:MountingHole_3.2mm_M3_DIN965, F.Cu at (125.0, 130.2)
- added REF**: MountingHole_3.2mm_M3_DIN965, Mounting_Holes:MountingHole_3.2mm_M3_DIN965, F.Cu at (57.5, 85.7)
- added REF**: MountingHole_3.2mm_M3_DIN965, Mounting_Holes:MountingHole_3.2mm_M3_DIN965, F.Cu at (142.5, 85.7)
- added REF**: MountingHole_3.2mm_M3_DIN965, Mounting_Holes:MountingHole_3.2mm_M3_DIN965, F.Cu at (57.5, 114.3)
- added REF**: MountingHole_3.2mm_M3_DIN965, Mounting_Holes:MountingHole_3.2mm_M3_DIN965, F.Cu at (142.5, 114.3)
- added U2: DA108S1, SMD_Packages:SOIC-8-N, F.Cu at (117.2, 107.2)
- added U3: DA108S1, SMD_Packages:SOIC-8-N, F.Cu at (135.6, 93.8)
- added U4: DA108S1, SMD_Packages:SOIC-8-N, F.Cu at (135.8, 106.5)
- added U5: DA108S1, SMD_Packages:SOIC-8-N, F.Cu at (260.2, 88.0)
- M1: footprint Socket_Strips:Socket_Strip_Straight_2x18_Pitch2.54mm -> pcb:particle_electron
- R1, R2, R3, R4: value R -> 10K
- R10, R11, R12, R9: value R -> 4.75K
- R13, R14, R15, R16, R25, R26, R27, R28, R37, R38, R39, R40: value R -> 47K
- R29, R30, R31, R32, R33, R34, R35, R36: value R -> 1K
- U1: value 7805 -> DA108S1; footprint Power_Integrations:TO-220 -> SMD_Packages:SOIC-8-N
- moved M1 129.7 mm to (75.0, 100.0), turned to 180 degrees
- moved P1 90.0 mm to (125.6, 87.6)
- moved R36 69.2 mm to (225.2, 44.0)
- moved R25 66.5 mm to (182.8, 145.0)
- moved R6 64.2 mm to (202.2, 54.8)
- moved R12 64.2 mm to (207.5, 55.3)
- moved R34 63.2 mm to (218.2, 38.5)
- moved R35 63.2 mm to (218.2, 41.8)
- moved R32 61.3 mm to (182.8, 143.0), turned to 180 degrees
- moved R31 57.6 mm to (182.5, 136.5), turned to 180 degrees
- moved R26 57.0 mm to (182.5, 138.5)
- moved Q1 53.0 mm to (189.2, 122.2)
- moved Q2 49.1 mm to (188.5, 129.0)
- moved R27 45.3 mm to (183.0, 130.0)
- moved R28 35.9 mm to (184.3, 123.2)
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Connections:
- M1 pad 10: Net-(C5-Pad1) -> Net-(M1-Pad10)
- M1 pad 11: Net-(C4-Pad1) -> Net-(M1-Pad11)
- M1 pad 12: Net-(C3-Pad1) -> Net-(M1-Pad12)
- M1 pad 5: Net-(C10-Pad1) -> Net-(M1-Pad5)
- M1 pad 6: Net-(C9-Pad1) -> Net-(M1-Pad6)
- M1 pad 7: Net-(C8-Pad1) -> Net-(M1-Pad7)
- M1 pad 8: Net-(C7-Pad1) -> Net-(M1-Pad8)
- M1 pad 9: Net-(C6-Pad1) -> Net-(M1-Pad9)
- Q1 pad 3: Net-(Q1-Pad3) -> /12V_OUT_3
- Q2 pad 3: Net-(Q2-Pad3) -> /12V_OUT_2
- Q3 pad 3: Net-(Q3-Pad3) -> /12V_OUT_1
- Q4 pad 3: Net-(Q4-Pad3) -> /12V_OUT_0
- R1 pad 1: Net-(R1-Pad1) -> Net-(M1-Pad5)
- R10 pad 1: Net-(R10-Pad1) -> Net-(M1-Pad11)
- R11 pad 1: Net-(R11-Pad1) -> Net-(M1-Pad10)
- R12 pad 1: Net-(R12-Pad1) -> Net-(M1-Pad9)
- R13 pad 1: Net-(R13-Pad1) -> Net-(M1-Pad8)
- R14 pad 1: Net-(R14-Pad1) -> Net-(M1-Pad7)
- R15 pad 1: Net-(R15-Pad1) -> Net-(M1-Pad6)
- R16 pad 1: Net-(R1-Pad1) -> Net-(M1-Pad5)
- R2 pad 1: Net-(R15-Pad1) -> Net-(M1-Pad6)
- R3 pad 1: Net-(R14-Pad1) -> Net-(M1-Pad7)
- R4 pad 1: Net-(R13-Pad1) -> Net-(M1-Pad8)
- R5 pad 1: Net-(R12-Pad1) -> Net-(M1-Pad9)
- R6 pad 1: Net-(R11-Pad1) -> Net-(M1-Pad10)
- R7 pad 1: Net-(R10-Pad1) -> Net-(M1-Pad11)
- R8 pad 1: Net-(R24-Pad2) -> Net-(M1-Pad12)
- R9 pad 1: Net-(R24-Pad2) -> Net-(M1-Pad12)
- U1 pad 1: (no net) -> /VSENSE_3
- U1 pad 2: (no net) -> /VSENSE_2
- U1 pad 3: (no net) -> /VSENSE_1
Other:
- board outline added: 104 x 79 mm
